File: WMD_Board/WMD_Board.sch (EAGLE design)
At the start: 0 parts

Commit message: Added algorithm chip
Parts:
- added C2, C3, C4: 1uF, SparkFun-Capacitors:1.0UF-0603-16V-10%
- added C5: 100nF, SparkFun-Capacitors:1.0UF-0603-16V-10%
- added R4, R5: 4.7k, SparkFun-Resistors:100KOHM-0603-1/10W-1%
- added R6: 10, SparkFun-Resistors:100KOHM-0603-1/10W-1%
- added U$1: MAX32664_TQFN, MAX32664:MAX32664_TQFN
- added Y1: ABS06-107-32.768KHZ-T, ABS06-107-32.768KHZ-T:ABS06-107-32.768KHZ-T
Connections:
- new net 1.8SCL_MICRO: R5.1, U$1.SLAVE_SCL
- new net 1.8SDA_MICRO: R4.1, U$1.SLAVE_SDA
- new net 1.8V: C2.1, C3.1, R4.2, R5.2, U$1.VDD@1, U$1.VDD@2
- new net GND: C2.2, C3.2, C4.1, R6.1, U$1.EP, U$1.VSS@1, U$1.VSS@2
- new net HR_SCL: U$1.SENSOR_SCL
- new net HR_SDA: U$1.SENSOR_SDA
- new net INT: U$1.HR_INT
- new net MFIO: U$1.MFIO
- new net N$1: U$1.32KIN, Y1.2
- new net N$3: U$1.32KOUT, Y1.1
- new net N$4: C4.2, U$1.VCORE
- new net N$7: C5.2, R6.2
- new net RSTN: C5.1, U$1.RSTN

Commit message: Schematic Progress
Parts:
- added C1, C15, C7, C9: 0.1uF, SparkFun-Capacitors:0.1UF-0603-25V-(+80/-20%)
- added C10, C16, C6, C8: 1.0uF, SparkFun-Capacitors:1.0UF-0603-16V-10%
- added C11: 10uF, SparkFun-Capacitors:10UF-0603-6.3V-20%
- added C17: 4.7uF, SparkFun-Capacitors:4.7UF0603
- added J4: EMPCB.SMAFSTJ.B.HT, EMPCB.SMAFSTJ.B.HT:EMPCB.SMAFSTJ.B.HT
- added JP2: (no value), microbuilder:HEADER-1X1ROUND
- added LED1: (no value), led:LEDCHIP-LED0805
- added R1, R2: 1k, SparkFun-Resistors:1KOHM-0603-1/10W-1%
- added RESET: SWITCH, DiscreteComponents:SWITCH
- added SV2: (no value), con-lsta:FE05-1
- added U1: STM32L053C8T6, STM32L053C8T6:STM32L053C8T6
- added U2: RFM69HCW, microbuilder:RFM69HCW_SMT
Connections:
- new net 3.3V: C1.1, C10.1, C11.1, C15.1, C16.1, C6.1, C7.1, C8.1, C9.1, R1.2, SV2.5, U1.VDD, U1.VDDA, U1.VDD_USB, U2.VDD
- new net CS: U1.PA4, U2.NSS
- new net DIO0: U1.PB1, U2.DIO0
- new net DIO1: U2.DIO1
- new net DIO2: U2.DIO2
- new net DIO3: U2.DIO3
- new net DIO4: U2.DIO4
- new net DIO5: U2.DIO5
- new net N$2: R2.2, U1.PB12
- new net N$5: LED1.A, R2.1
- new net N$6: J4.1, JP2.1, U2.ANT
- new net NRST: C17.1, R1.1, RESET.P$2, SV2.1, U1.NRST
- new net OSC_IN: U1.PH0-OSC_IN
- new net OSC_OUT: U1.PH1-OSC_OUT
- new net RST: U1.PB0, U2.RESET
- new net SPI1_MISO: U1.PA6, U2.MISO
- new net SPI1_MOSI: U1.PA7, U2.MOSI
- new net SPI1_SCK: U1.PA5, U2.SCK
- new net SWCLK: SV2.4, U1.PA14
- new net SWDIO: SV2.2, U1.PA13
- new net USB_DM_3V3: U1.PA11
- new net USB_DP_3V3: U1.PA12
- net GND: now also C1.2, C10.2, C11.2, C15.2, C16.2, C17.2, C6.2, C7.2, C8.2, C9.2, J4.2, LED1.C, RESET.P$1, SV2.3, U1.VSS, U1.VSSA, U2.GND@1, U2.GND@2, U2.GND@3
Other:
- note added: "Heart-Rate Algorithm Chip"
- note added: "LoRa Module"
- note added: "PROGRAMMING HEADER"
- note added: "STM32L0"

Commit message: Schematic
Parts:
- removed C2, C3, C4: 1uF, SparkFun-Capacitors:1.0UF-0603-16V-10%
- removed C5: 100nF, SparkFun-Capacitors:1.0UF-0603-16V-10%
- removed J4: EMPCB.SMAFSTJ.B.HT, EMPCB.SMAFSTJ.B.HT:EMPCB.SMAFSTJ.B.HT
- removed JP2: (no value), microbuilder:HEADER-1X1ROUND
- removed R4, R5: 4.7k, SparkFun-Resistors:100KOHM-0603-1/10W-1%
- removed R6: 10, SparkFun-Resistors:100KOHM-0603-1/10W-1%
- removed U$1: MAX32664_TQFN, MAX32664:MAX32664_TQFN
- removed U2: RFM69HCW, microbuilder:RFM69HCW_SMT
- removed Y1: ABS06-107-32.768KHZ-T, ABS06-107-32.768KHZ-T:ABS06-107-32.768KHZ-T
- added C12: 10uF, SparkFun-Capacitors:10UF-0603-6.3V-20%
- added C13, C18: 1uF, SparkFun-Capacitors:1.0UF-0603-16V-10%
- added C14: 100nF, SparkFun-Capacitors:1.0UF-0603-16V-10%
- added J1: EMPCB.SMAFSTJ.B.HT, EMPCB.SMAFSTJ.B.HT:EMPCB.SMAFSTJ.B.HT
- added JP1: (no value), microbuilder:HEADER-1X1ROUND
- added R3: 10, SparkFun-Resistors:100KOHM-0603-1/10W-1%
- added R7, R8: 4.7k, SparkFun-Resistors:100KOHM-0603-1/10W-1%
- added U$10: MAX32664_TQFN, MAX32664:MAX32664_TQFN
- added U3: RFM69HCW, microbuilder:RFM69HCW_SMT
- added Y2: ABS06-107-32.768KHZ-T, ABS06-107-32.768KHZ-T:ABS06-107-32.768KHZ-T
- C11: value 10uF -> 1uF; device SparkFun-Capacitors:10UF-0603-6.3V-20% -> SparkFun-Capacitors:1.0UF-0603-16V-10%
Connections:
- removed net 1.8SCL_MICRO: R5.1, U$1.SLAVE_SCL
- removed net 1.8SDA_MICRO: R4.1, U$1.SLAVE_SDA
- removed net HR_SCL: U$1.SENSOR_SCL
- removed net HR_SDA: U$1.SENSOR_SDA
- removed net N$1: U$1.32KIN, Y1.2
- removed net N$3: U$1.32KOUT, Y1.1
- removed net N$4: C4.2, U$1.VCORE
- removed net N$7: C5.2, R6.2
- removed net OSC_IN: U1.PH0-OSC_IN
- removed net OSC_OUT: U1.PH1-OSC_OUT
- removed net USB_DM_3V3: U1.PA11
- removed net USB_DP_3V3: U1.PA12
- new net GPS_RX: U1.PB11
- new net GPS_TX: U1.PB10
- new net N$10: U$10.32KIN, Y2.2
- new net N$11: U$10.32KOUT, Y2.1
- new net N$8: J1.1, JP1.1, U3.ANT
- new net N$9: C14.2, R3.2
- new net SCL_EEPROM: U1.PB13
- new net SCL_HR: U1.PB6
- new net SCL_HR_1.8V: R8.1, U$10.SLAVE_SCL
- new net SCL_TO_HR_SENSOR: U$10.SENSOR_SCL
- new net SDA_EEPROM: U1.PB14
- new net SDA_HR: U1.PB7
- new net SDA_HR_1.8V: R7.1, U$10.SLAVE_SDA
- new net SDA_TO_HR_SENSOR: U$10.SENSOR_SDA
- net 1.8V: now also C11.1, C18.1, R7.2, R8.2, U$10.VDD@1, U$10.VDD@2; no longer C2.1, C3.1, R4.2, R5.2, U$1.VDD@1, U$1.VDD@2
- net 3.3V: now also C12.1, U3.VDD; no longer C11.1, U2.VDD
- net CS: now also U3.NSS; no longer U2.NSS
- net DIO0: now also U3.DIO0; no longer U2.DIO0
- net DIO1: now also U3.DIO1; no longer U2.DIO1
- net DIO2: now also U3.DIO2; no longer U2.DIO2
- net DIO3: now also U3.DIO3; no longer U2.DIO3
- net DIO4: now also U3.DIO4; no longer U2.DIO4
- net DIO5: now also U3.DIO5; no longer U2.DIO5
- net GND: now also C12.2, C13.1, C18.2, J1.2, R3.1, U$10.EP, U$10.VSS@1, U$10.VSS@2, U3.GND@1, U3.GND@2, U3.GND@3; no longer C2.2, C3.2, C4.1, J4.2, R6.1, U$1.EP, U$1.VSS@1, U$1.VSS@2, U2.GND@1, U2.GND@2, U2.GND@3
- net INT: now also U$10.HR_INT; no longer U$1.HR_INT
- net MFIO: now also U$10.MFIO; no longer U$1.MFIO
- net N$6: now also C13.2, U$10.VCORE; no longer J4.1, JP2.1, U2.ANT
- net RST: now also U3.RESET; no longer U2.RESET
- net RSTN: now also C14.1, U$10.RSTN; no longer C5.1, U$1.RSTN
- net SPI1_MISO: now also U3.MISO; no longer U2.MISO
- net SPI1_MOSI: now also U3.MOSI; no longer U2.MOSI
- net SPI1_SCK: now also U3.SCK; no longer U2.SCK

Commit message: More Schematic Work
Parts:
- removed R7, R8: 4.7k, SparkFun-Resistors:100KOHM-0603-1/10W-1%
- added R4, R5, R6, R9: 4.7k, SparkFun-Resistors:1KOHM-0603-1/10W-1%
- added U2, U4: BSS138, BSS138:BSS138
Connections:
- net 1.8V: now also R4.2, R6.2, U2.G, U4.G; no longer R7.2, R8.2
- net 3.3V: now also R5.1, R9.1
- net SCL_HR: now also R9.2, U4.D
- net SCL_HR_1.8V: now also R6.1, U4.S; no longer R8.1
- net SDA_HR: now also R5.2, U2.D
- net SDA_HR_1.8V: now also R4.1, U2.S; no longer R7.1
Other:
- note added: "Logic Level Conversion for Heart-Rate I2C"
